File: MartinSM850DMXReceiverSchematics/MartinSM850DMXReceiverSchematics.kicad_sch (KiCad schematic)
At the start: 11 parts, among them J1 DMX_Socket

Commit message: Updated README and added Schematics and User manual
Parts:
- added DIN_Ready_LED1: Green, symbol Device:LED
- added DIN_Socket1: DIN_Socket, symbol Connector:Conn_01x05_Socket
- added Fogging_LED1: White, symbol Device:LED
- added Fogging_LED_Resistor1, Fogging_Transistor_Resistor1: 220 Ohm, symbol Device:R
- added Fogging_Transistor1: S8050, Package_TO_SOT_THT:TO-92_Inline, symbol Transistor_BJT:S8050
- DMX_Socket_In1: renamed from DMX_Socket; value DMX -> DMX_Socket_In
- DMX_Socket_Out1: renamed from J1; value DMX_Socket -> DMX_Socket_Out
- renumbered Address_Switches to Address_Switches1, Address_Valid_LED_Resistor to Address_Valid_LED_Resistor1, Arduino_Pro_Mini to Arduino_Pro_Mini1, Coupling_Capacitor to Coupling_Capacitor1, Power_LED to Power_LED1, Power_LED_Resistor to Power_LED_Resistor1, RS485_Decoder to RS485_Decoder1, Termination_Resistor to Termination_Resistor1, Valid_Address_LED to Valid_Address_LED1
Connections:
- net GND: now also DIN_Ready_LED1.1 (K), DIN_Socket1.5 (Pin_5), Fogging_LED_Resistor1.2, Fogging_Transistor1.1 (E)
- net VCC: now also DIN_Socket1.2 (Pin_2)
- net D8: now reaches Arduino_Pro_Mini1.D8
- net D8: now also Fogging_LED1.2 (A), Fogging_Transistor_Resistor1.2
- new net: Fogging_Transistor1.2 (B), Fogging_Transistor_Resistor1.1
- new net: DIN_Socket1.4 (Pin_4), Fogging_Transistor1.3 (C)
- new net: Fogging_LED1.1 (K), Fogging_LED_Resistor1.1
- new net: DIN_Ready_LED1.2 (A), DIN_Socket1.1 (Pin_1)

Commit message: BugFix: invalid DMX address does stop fogging now. + Small improvements in kicad
Parts:
- Address_Switches1: footprint (none) -> Button_Switch_SMD:SW_DIP_SPSTx10_Slide_9.78x27.58mm_W8.61mm_P2.54mm
- Address_Valid_LED_Resistor1, Fogging_Transistor_Resistor1, Power_LED_Resistor1, Termination_Resistor1: footprint (none) -> Resistor_THT:R_Array_SIP4
- Arduino_Pro_Mini1: footprint PCM_arduino-library:Arduino_Pro_Mini_Socket -> Module:Arduino_Nano
- Coupling_Capacitor1: footprint (none) -> Capacitor_THT:CP_Axial_L10.0mm_D4.5mm_P15.00mm_Horizontal
- DIN_Ready_LED1, Fogging_LED1, Fogging_LED_Resistor1, Power_LED1, Valid_Address_LED1: footprint (none) -> LED_THT:LED_D3.0mm_Horizontal_O1.27mm_Z2.0mm
- DIN_Socket1: footprint (none) -> Connector_PinSocket_1.00mm:PinSocket_1x05_P1.00mm_Vertical
- DMX_Socket_In1, DMX_Socket_Out1: footprint (none) -> Connector_PinSocket_1.00mm:PinSocket_1x03_P1.00mm_Vertical
- RS485_Decoder1: footprint (none) -> Socket:DIP_Socket-24_W4.3_W5.08_W7.62_W10.16_W10.9_3M_224-5248-00-0602J
Changed lines of the file:
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@@
 			)
 		)
-		(property "Footprint" ""
+		(property "Footprint" "Connector_PinSocket_1.00mm:PinSocket_1x03_P1.00mm_Vertical"
 			(at 34.29 158.75 0)
 			(effects
@@
 			)
 		)
-		(property "Footprint" ""
+		(property "Footprint" "Resistor_THT:R_Array_SIP4"
 			(at 203.2 38.862 90)
 			(effects
@@
 			)
 		)
-		(property "Footprint" ""
+		(property "Footprint" "LED_THT:LED_D3.0mm_Horizontal_O1.27mm_Z2.0mm"
 			(at 44.45 76.2 0)
 			(effects
@@
 			)
 		)
-		(property "Footprint" ""
+		(property "Footprint" "Connector_PinSocket_1.00mm:PinSocket_1x03_P1.00mm_Vertical"
 			(at 34.29 148.59 0)
 			(effects
@@
 			)
 		)
-		(property "Footprint" ""
+		(property "Footprint" "Socket:DIP_Socket-24_W4.3_W5.08_W7.62_W10.16_W10.9_3M_224-5248-00-0602J"
 			(at 82.55 137.16 0)
 			(effects
@@
 			)
 		)
-		(property "Footprint" ""
+		(property "Footprint" "LED_THT:LED_D3.0mm_Horizontal_O1.27mm_Z2.0mm"
 			(at 233.172 44.45 90)
 			(effects
@@
 			)
 		)
-		(property "Footprint" ""
+		(property "Footprint" "Connector_PinSocket_1.00mm:PinSocket_1x05_P1.00mm_Vertical"
 			(at 271.78 62.23 0)
 			(effects
@@
 			)
 		)
-		(property "Footprint" ""
+		(property "Footprint" "LED_THT:LED_D3.0mm_Horizontal_O1.27mm_Z2.0mm"
 			(at 257.81 49.53 0)
 			(effects
@@
 			)
 		)
-		(property "Footprint" ""
+		(property "Footprint" "LED_THT:LED_D3.0mm_Horizontal_O1.27mm_Z2.0mm"
 			(at 222.25 35.56 0)
 			(effects
@@
 			)
 		)
-		(property "Footprint" ""
+		(property "Footprint" "Button_Switch_SMD:SW_DIP_SPSTx10_Slide_9.78x27.58mm_W8.61mm_P2.54mm"
 			(at 50.8 50.8 0)
 			(effects
@@
 			)
 		)
-		(property "Footprint" ""
+		(property "Footprint" "Resistor_THT:R_Array_SIP4"
 			(at 66.802 153.67 90)
 			(effects
@@
 			)
 		)
-		(property "Footprint" "PCM_arduino-library:Arduino_Pro_Mini_Socket"
+		(property "Footprint" "Module:Arduino_Nano"
 			(at 127 104.14 0)
 			(effects
@@
 			)
 		)
-		(property "Footprint" ""
+		(property "Footprint" "Resistor_THT:R_Array_SIP4"
 			(at 55.88 77.978 90)
 			(effects
@@
 			)
 		)
-		(property "Footprint" ""
+		(property "Footprint" "Capacitor_THT:CP_Axial_L10.0mm_D4.5mm_P15.00mm_Horizontal"
 			(at 101.9048 149.86 0)
 			(effects
@@
 			)
 		)
-		(property "Footprint" ""
+		(property "Footprint" "Resistor_THT:R_Array_SIP4"
 			(at 170.18 137.922 90)
 			(effects
@@
 			)
 		)
-		(property "Footprint" ""
+		(property "Footprint" "LED_THT:LED_D3.0mm_Horizontal_O1.27mm_Z2.0mm"
 			(at 158.75 139.7 0)
 			(effects
